File: PCB_USB_NiMH_Charger.kicad_sch (KiCad schematic)
At the start: 53 parts, among them J1 USB_C_Receptacle_Simple, J2 Conn_02x01, Q1 2SA1015, Q2 2SB834, Q3 2SB834, Q4 2SB834, Q5 2SB834, U1 LM339, U2 S-812C33A_TO92

Commit message: Update BT1, BT2
BT1, BT2のフットプリントを秋月電子公開のデータシートに従って更新。
Parts:
- BT1, BT2: footprint Battery:BatteryHolder_Keystone_2466_1xAAA -> mylib:BatteryHolder_COMF_BH-411-4P24_1xAAA
Changed lines of the file:
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@@
       (effects (font (size 1.27 1.27)) (justify left))
     )
-    (property "Footprint" "Battery:BatteryHolder_Keystone_2466_1xAAA" (at 170.18 72.136 90)
+    (property "Footprint" "mylib:BatteryHolder_COMF_BH-411-4P24_1xAAA" (at 170.18 72.136 90)
       (effects (font (size 1.27 1.27)) hide)
     )
@@
       (effects (font (size 1.27 1.27)) (justify left))
     )
-    (property "Footprint" "Battery:BatteryHolder_Keystone_2466_1xAAA" (at 260.35 72.136 90)
-      (effects (font (size 1.27 1.27)) hide)
-    )
+    (property "Footprint" "mylib:BatteryHolder_COMF_BH-411-4P24_1xAAA" (at 260.35 72.136 90)
+      (effects (font (size 1.27 1.27)) hide)
+    )

Commit message: 抵抗値を変更
Parts:
- R11, R7: value 2k -> 2.7k
- R15, R19: value 2k -> 1.6k
Changed lines of the file:
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@@
       (effects (font (size 1.27 1.27)) (justify left))
     )
-    (property "Value" "2k" (at 250.19 141.605 0)
+    (property "Value" "1.6k" (at 250.19 141.605 0)
       (effects (font (size 1.27 1.27)) (justify left))
     )
@@
       (effects (font (size 1.27 1.27)) (justify left))
     )
-    (property "Value" "2k" (at 160.02 141.605 0)
+    (property "Value" "1.6k" (at 160.02 141.605 0)
       (effects (font (size 1.27 1.27)) (justify left))
     )
@@
       (effects (font (size 1.27 1.27)) (justify left))
     )
-    (property "Value" "2k" (at 160.02 65.405 0)
+    (property "Value" "2.7k" (at 160.02 65.405 0)
       (effects (font (size 1.27 1.27)) (justify left))
     )
@@
       (effects (font (size 1.27 1.27)) (justify left))
     )
-    (property "Value" "2k" (at 250.19 65.405 0)
-      (effects (font (size 1.27 1.27)) (justify left))
-    )
+    (property "Value" "2.7k" (at 250.19 65.405 0)
+      (effects (font (size 1.27 1.27)) (justify left))
+    )

Commit message: 半固定抵抗のフットプリントを修正
Parts:
- RV1: footprint Potentiometer_THT:Potentiometer_ACP_CA6-H2,5_Horizontal -> mylib:Potentiometer_TOCOS_GF063P_Vertical
Changed lines of the file:
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@@
       (effects (font (size 1.27 1.27)) (justify right))
     )
-    (property "Footprint" "Potentiometer_THT:Potentiometer_ACP_CA6-H2,5_Horizontal" (at 57.15 143.51 0)
+    (property "Footprint" "mylib:Potentiometer_TOCOS_GF063P_Vertical" (at 57.15 143.51 0)
       (effects (font (size 1.27 1.27)) hide)
     )
